File: A2VGA.v1.6-hardware/A2VGA.v1.6.kicad_sch (KiCad schematic)
At the start: 40 parts, among them CON1 Apple2_edge_connector, CON2 VGA DB15_Female, Q1 BS170, U1 RPI-Pico, U2 74LVC245, U3 74LVC245, U4 74LVC245, U5 ATF22V10C

Commit message: Add files via upload
Parts:
- removed Q1: BS170, Package_TO_SOT_THT:TO-92_Inline, symbol Transistor_FET:BS170
- added Q1: 2N7000, Package_TO_SOT_THT:TO-92_Inline, symbol Transistor_FET:2N7000
Connections:
- net GND: now also Q1.1 (S)
- net at R18.1, R19.1: now also Q1.2 (G)
- net at CON1.30 (~{IRQ}): now also Q1.3 (D)
