File: A2VGA.v1.6-hardware/A2VGA.v1.6.kicad_pcb (KiCad board)
At the start: 2 copper layers, 99.7 x 61.4 mm, 90 parts, among them CON2 DB15_Female_HighDensity_Mount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, Q1 TO-92L_Inline_Wide, U1 Pico / PicoW, U2 74LVC245, U3 74LVC245, U4 74LVC245, U5 ATF22V10

Commit message: Add files via upload
Parts:
- Q1: value TO-92L_Inline_Wide -> 2N7000
- moved Q1 5.16 mm to (107.0, 112.0), turned to 0 degrees
Connections:
- Q1 pad 1: IRQ -> GND
- Q1 pad 3: GND -> IRQ

Commit message: Add files via upload
Routing:
- net GND: track 163.1 -> 171.3 mm
- net IRQ: track 74.1 -> 72.2 mm, vias 4 -> 3
Changed lines of the file:
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@@
 		(tags "TO-92L Inline Wide transistor")
 		(property "Reference" "Q1"
-			(at -1.6764 -2.0066 360)
+			(at -1.6764 -2.0066 0)
 			(layer "F.SilkS")
 			(effects
@@
 		)
 		(property "Value" "2N7000"
-			(at 2.54 2.79 360)
+			(at 2.54 2.79 0)
 			(layer "F.Fab")
 			(effects
@@
 		)
 		(property "Footprint" ""
-			(at 0 0 360)
+			(at 0 0 0)
 			(layer "F.Fab")
 			(hide yes)
@@
 		)
 		(property "Datasheet" ""
-			(at 0 0 360)
+			(at 0 0 0)
 			(layer "F.Fab")
 			(hide yes)
@@
 		)
 		(property "Description" ""
-			(at 0 0 360)
+			(at 0 0 0)
 			(layer "F.Fab")
 			(hide yes)
@@
 		)
 		(fp_text user "${REFERENCE}"
-			(at 2.54 0 360)
+			(at 2.54 0 0)
 			(layer "F.Fab")
 			(effects
@@
 	)
 	(segment
+		(start 116.1288 117.0432)
+		(end 116.1288 118.4148)
+		(width 0.25)
+		(layer "F.Cu")
+		(net 1)
+	)
+	(segment
 		(start 92.272165 109.214)
 		(end 93.107165 109.214)
@@
 	)
 	(segment
+		(start 115.2906 116.205)
+		(end 116.1288 117.0432)
+		(width 0.25)
+		(layer "F.Cu")
+		(net 1)
+	)
+	(segment
+		(start 116.1288 118.4148)
+		(end 116.459 118.745)
+		(width 0.25)
+		(layer "F.Cu")
+		(net 1)
+	)
+	(segment
 		(start 92.272165 109.214)
 		(end 92.272165 106.972669)
@@
 		(net 1)
 	)
+	(segment
+		(start 118.11 112.141)
+		(end 115.2906 114.9604)
+		(width 0.25)
+		(layer "F.Cu")
+		(net 1)
+	)
+	(segment
+		(start 115.2906 114.9604)
+		(end 115.2906 116.205)
+		(width 0.25)
+		(layer "F.Cu")
+		(net 1)
+	)
 	(via
 		(at 133.604 83.439)
@@
 	)
 	(via
-		(at 114.173 118.491)
+		(at 114.4016 118.3894)
 		(size 0.8)
 		(drill 0.4)
@@
 	)
 	(via
-		(at 114.173 117.602)
+		(at 114.3508 117.7036)
 		(size 0.8)
 		(drill 0.4)
@@
 	)
 	(segment
+		(start 115.3414 123.0747)
+		(end 116.7892 124.5225)
+		(width 0.2)
+		(layer "F.Cu")
+		(net 70)
+	)
+	(segment
+		(start 112.014 112.014)
+		(end 112.014 112.920214)
+		(width 0.2)
+		(layer "F.Cu")
+		(net 70)
+	)
+	(segment
+		(start 114.634293 115.540507)
+		(end 114.634293 116.742493)
+		(width 0.2)
+		(layer "F.Cu")
+		(net 70)
+	)
+	(segment
 		(start 161.29 129.54)
 		(end 161.29 126.111)
@@
 	)
 	(segment
-		(start 115.189 112.014)
-		(end 112.014 112.014)
+		(start 115.3414 117.4496)
+		(end 115.3414 123.0747)
 		(width 0.2)
 		(layer "F.Cu")
@@
 	)
 	(segment
-		(start 115.189 122.9223)
-		(end 115.189 112.014)
+		(start 112.014 112.920214)
+		(end 114.634293 115.540507)
 		(width 0.2)
 		(layer "F.Cu")
@@
 	)
 	(segment
-		(start 116.7892 124.5225)
-		(end 115.189 122.9223)
+		(start 114.634293 116.742493)
+		(end 115.3414 117.4496)
 		(width 0.2)
 		(layer "F.Cu")
 		(net 70)
 	)
-	(via
-		(at 115.189 112.014)
-		(size 0.8)
-		(drill 0.4)
-		(layers "F.Cu" "B.Cu")
-		(net 70)
-	)
